File: Farkas/Sebessegmero.kicad_pcb (KiCad board)
At the start: 2 copper layers, 47 x 50.8 mm, 32 parts, among them J1 Conn_01x02_Female, J2 Conn_01x02_Female, J3 Screw_Terminal_01x02, J4 Conn_02x04_Odd_Even, J5 Conn_01x03_Female, U1 Opamp_Quad_Generic

Commit message: kesz aramkor
Parts:
- added M3: MountingHole_3.2mm_M3, MountingHole:MountingHole_3.2mm_M3, F.Cu at (53.3, 77.5)
- moved J3 5.24 mm to (69.8, 74.9)
- moved C1 5.24 mm to (80.3, 68.1)
- moved R15 5.24 mm to (87.6, 55.9)
- moved R16 5.24 mm to (87.6, 58.8)
- moved R18 5.24 mm to (87.6, 52.6)
- moved R5 5.24 mm to (69.7, 51.4)
- moved J4 5.24 mm to (76.8, 32.9)
- moved R21 5.24 mm to (87.5, 45.6)
- moved R22 5.24 mm to (84.5, 45.6)
- moved U1 5.24 mm to (80.0, 53.3)
- moved J1 5.24 mm to (86.5, 66.5)
- moved J5 5.24 mm to (69.8, 34.3)
- moved M3 5.24 mm to (87.6, 77.5)
- moved R11 5.24 mm to (69.8, 45.7)
- moved R17 5.24 mm to (87.6, 61.7)
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- renumbered REF** to M3
Routing:
- net Net-(J2-Pad1): track 15.7 -> 33.4 mm
- net GND: vias 4 -> 11
Other:
- outline, holes or cut-outs redrawn
- board text added: "FONP0O"

Commit message: doksi 3.0
Parts:
- moved J2 0.64 mm to (87.0, 35.4)
- moved J5 0.38 mm to (69.8, 34.7)
- moved J1 0.25 mm to (86.7, 66.5)
Routing:
- net Net-(J2-Pad1): track 33.4 -> 31.7 mm
Other:
- board text added: "10V"
- board text added: "12V"
- board text added: "20mA"
- board text added: "3V3"
- board text added: "4-"
- board text added: "5V"
- board text added: "AN_IN"
- board text added: "AN_OUT"
- board text added: "GND"
- board text added: "I2C"
